File: 2017MXP/2017MXP board.brd (EAGLE design)
At the start: 73.3 x 80 mm, 50 parts, among them U1 ATMEGA328P, U3 ATMEGA328P, X1 057-034-1, Y1 16MHz, Y2 16MHz

Commit message: Updated the boards for final layout.
Parts:
- added R12, R13: 10k, SparkFun-Passives:0603-RES
Connections:
- removed net N$13: U3.13
- net LED-D9: now also U3.13
- net SCL: now also R13.1
- net SDA: now also R12.1
- net VCC: now also R12.2, R13.2
Routing:
- net SDA: track 97.2 -> 156.3 mm, vias 3 -> 4
- net SCL: track 67.6 -> 107.4 mm
- net SCL3.3: track 82.0 -> 117.3 mm
- net LED-D9: track 0.00 -> 22.7 mm
- net LED-D8: track 46.3 -> 25.9 mm, vias 2 -> 3
- net LED-SCK: track 35.9 -> 54.7 mm, vias 4 -> 2
- net LED-MISO: track 64.8 -> 48.1 mm, vias 1 -> 3
- net LED-RESET: track 119.7 -> 103.4 mm, vias 3 -> 4
- net GND: track 470.4 -> 459.3 mm
- net LED-D10: track 31.7 -> 38.6 mm, vias 0 -> 2
- net VCC: track 248.8 -> 244.6 mm, vias 4 -> 5
- net LED-MOSI: track 49.8 -> 45.8 mm, vias 2 -> 1
- net LED-D6: track 32.9 -> 35.1 mm, vias 1 -> 2
- net LED-D3: track 23.3 -> 22.4 mm
- net LED-D5: track 26.9 -> 26.7 mm, vias 2 -> 3
Other:
- outline, holes or cut-outs redrawn
