File: 2017MXP/2017MXP board.sch (EAGLE design)
At the start: 50 parts, among them U1 ATMEGA328P, U3 ATMEGA328P, X1 057-034-1, Y1 16MHz, Y2 16MHz

Commit message: Updated the boards for final layout.
Parts:
- added R12, R13: 10k, SparkFun-Passives:RESISTOR0603-RES
Connections:
- removed net N$13: U3.PB1(OC1A)
- net LED-D9: now also U3.PB1(OC1A)
- net SCL: now also R13.1
- net SDA: now also R12.1
- net VCC: now also R12.2, R13.2
Changed lines of the file:
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@@
 <?xml version="1.0" encoding="utf-8"?>
 <!DOCTYPE eagle SYSTEM "eagle.dtd">
-<eagle version="7.2.0">
+<eagle version="7.1.0">
 <drawing>
 <settings>
@@
 <part name="U$2" library="LSF-SMT" deviceset="LSF-SMT" device=""/>
 <part name="X1" library="con-panduit" deviceset="057-034-" device="1"/>
+<part name="R12" library="SparkFun-Passives" deviceset="RESISTOR" device="0603-RES" value="10k"/>
+<part name="R13" library="SparkFun-Passives" deviceset="RESISTOR" device="0603-RES" value="10k"/>
+<part name="SUPPLY10" library="SparkFun-Aesthetics" deviceset="VCC" device=""/>
+<part name="SUPPLY12" library="SparkFun-Aesthetics" deviceset="VCC" device=""/>
 </parts>
 <sheets>
@@
 <instance part="X1" gate="-33" x="1536.7" y="287.02"/>
 <instance part="X1" gate="-34" x="1559.56" y="287.02"/>
+<instance part="R12" gate="G$1" x="1706.88" y="330.2" rot="R90"/>
+<instance part="R13" gate="G$1" x="1722.12" y="330.2" rot="R90"/>
+<instance part="SUPPLY10" gate="G$1" x="1706.88" y="340.36"/>
+<instance part="SUPPLY12" gate="G$1" x="1722.12" y="340.36"/>
 </instances>
 <busses>
@@
 <label x="1518.92" y="368.3" size="1.778" layer="95" rot="R180" xref="yes"/>
 </segment>
+<segment>
+<pinref part="R12" gate="G$1" pin="2"/>
+<pinref part="SUPPLY10" gate="G$1" pin="VCC"/>
+<wire x1="1706.88" y1="340.36" x2="1706.88" y2="335.28" width="0.1524" layer="91"/>
+</segment>
+<segment>
+<pinref part="R13" gate="G$1" pin="2"/>
+<pinref part="SUPPLY12" gate="G$1" pin="VCC"/>
+<wire x1="1722.12" y1="340.36" x2="1722.12" y2="335.28" width="0.1524" layer="91"/>
+</segment>
 </net>
 <net name="RXI" class="0">
@@
 <label x="1877.06" y="251.46" size="1.27" layer="95" xref="yes"/>
 </segment>
+<segment>
+<pinref part="R12" gate="G$1" pin="1"/>
+<wire x1="1706.88" y1="325.12" x2="1706.88" y2="317.5" width="0.1524" layer="91"/>
+</segment>
 </net>
 <net name="SCL" class="0">
@@
 <wire x1="1871.98" y1="248.92" x2="1877.06" y2="248.92" width="0.1524" layer="91"/>
 <label x="1877.06" y="248.92" size="1.27" layer="95" xref="yes"/>
+</segment>
+<segment>
+<pinref part="R13" gate="G$1" pin="1"/>
+<wire x1="1722.12" y1="325.12" x2="1722.12" y2="317.5" width="0.1524" layer="91"/>
 </segment>
 </net>
@@
 <pinref part="JP18" gate="G$1" pin="4"/>
 </segment>
+<segment>
+<pinref part="U3" gate="G$1" pin="PB1(OC1A)"/>
+<wire x1="1871.98" y1="213.36" x2="1877.06" y2="213.36" width="0.1524" layer="91"/>
+</segment>
 </net>
 <net name="LED-D10" class="0">
@@
 </segment>
 </net>
-<net name="N$13" class="0">
-<segment>
-<pinref part="U3" gate="G$1" pin="PB1(OC1A)"/>
-<wire x1="1871.98" y1="213.36" x2="1877.06" y2="213.36" width="0.1524" layer="91"/>
-</segment>
-</net>
