File: Ringlight board/RingLight.brd (EAGLE design)
At the start: 44.8 x 44.4 mm, 17 parts, among them P1 M-1X02-SIP-100-32Y

Commit message: Updated the boards for final layout.
Routing:
- net VCC: track 129.3 -> 105.9 mm, vias 3 -> 0
- net N$8: track 21.8 -> 10.9 mm
- net GND: track 118.0 -> 107.6 mm
- net N$6: track 13.6 -> 11.5 mm, vias 2 -> 0
- net N$10: track 17.3 -> 18.3 mm, vias 2 -> 0
- net N$7: track 16.5 -> 17.4 mm, vias 2 -> 0
- net N$1: track 11.8 -> 12.7 mm, vias 2 -> 0
- net N$2: track 7.47 -> 6.71 mm, vias 0 -> 2
- net N$5: track 12.4 -> 11.9 mm
Other:
- outline, holes or cut-outs redrawn
- board text added: "+12v"
- board text added: "CUT OUT"
- board text added: "GND"
- board text removed: "VCC"
